File: emberone.kicad_pcb (KiCad board)
At the start: 6 copper layers, 125 x 125 mm, 409 parts, among them J1 Screw Terminal, J10 Conn_01x01, J11 Conn_01x01, J14 Conn_01x01, J15 Conn_01x01, J18 Conn_01x01, J19 Conn_Coaxial, J2 Screw Terminal, J20 Conn_01x06, J21 Conn_01x01, J3 Conn_01x01, J4 Conn_01x01, J5 Conn_01x01, J6 USB_C_Receptacle_USB2.0, J7 Conn_01x01, J8 Conn_01x01, J9 Conn_01x01, Q1 CSD18511Q5A, Q2 CSD18511Q5A, Q3 CSD18511Q5A, Q4 CSD18511Q5A, Q5 NVMFS5C645NLAFT1G, SW1 GT-TC029B-H025-L1N, SW2 GT-TC029B-H025-L1N, U1 LM25119PSQ/NOPB, U10 TLV1117LV33DCYR, U11 TPD1E05U06DYA, U12 TPD1E05U06DYA, U13 TMP451HQDQWRQ1, U2 DS4432U+, U27 RP2040, U28 MCP1824T-1202E/OT, U29 MCP1824T-1202E/OT, U3 INA260, U30 MCP1824T-1202E/OT, U32 MCP1824T-0802E, U4 SN74AVC4T774, U42 MCP1824T-0802E, U43 MCP1824T-0802E, U45 BM1362AC_MODE1, U46 BM1362AC_MODE0, U47 BM1362AC_MODE1, U48 MCP1824T-1202E/OT, U49 MCP1824T-1202E/OT, U5 25MHz, U50 MCP1824T-1202E/OT, U51 MCP1824T-0802E, U52 MCP1824T-0802E, U53 MCP1824T-0802E, U54 BM1362AC_MODE1, U55 BM1362AC_MODE0, U56 BM1362AC_MODE1, U57 MCP1824T-1202E/OT, U58 MCP1824T-1202E/OT, U59 MCP1824T-1202E/OT, U6 TMP1075, U60 MCP1824T-0802E, U61 MCP1824T-0802E, U62 MCP1824T-0802E, U63 BM1362AC_MODE1, U64 BM1362AC_MODE0, U65 BM1362AC_MODE1, U66 MCP1824T-1202E/OT, U67 MCP1824T-1202E/OT, U68 MCP1824T-1202E/OT, U69 MCP1824T-0802E, U7 AP74700Q, U70 MCP1824T-0802E, U71 MCP1824T-0802E, U72 BM1362AC_MODE1, U73 BM1362AC_MODE0, U74 BM1362AC_MODE1, U8 W25Q16JVUXIQ TR, U9 SK6812, Y1 12MHz

Commit message: remover old gerbers, bom, ibom. Changed C29 to 1000pF for #47
Parts:
- C29: value 4700pF -> 1000pF
- R34: value 50k -> 49.9k
- R61, R70: value 50 -> 49.9
